Commit message: c

File: lebai_lm3_support/urdf/gripper_macro.xacro (robot description, xacro)
@@ -117,5 +117,5 @@
 <!-- end of link list -->
 <!-- joint list -->
-<joint name="${prefix}gripper_r_joint1" type="revolute">
+<joint name="${prefix}gripper_r_joint1" type="fixed">
 	<parent link="${prefix}gripper_base_link"/>
 	<child link="${prefix}gripper_r_link1"/>
@@ -124,19 +124,19 @@
 	<limit lower="-10.0" upper="10.0" effort="100" velocity="1" />
 </joint>
-<joint name="${prefix}gripper_r_joint2" type="revolute">
+<joint name="${prefix}gripper_r_joint2" type="fixed">
 	<parent link="${prefix}gripper_base_link"/>
 	<child link="${prefix}gripper_r_link2"/>
-        <origin xyz="0.0115 0.0 0.1056" rpy="${PI_2} 0 0"/>
+	<origin xyz="0.0115 0.0 0.1056" rpy="${PI_2} 0 0"/>
 	<axis xyz="0 0 1" />
 	<limit lower="-10.0" upper="10.0" effort="100" velocity="1" />
 </joint>
-<joint name="${prefix}gripper_r_joint_finger" type="revolute">
+<joint name="${prefix}gripper_r_joint_finger" type="fixed">
 	<parent link="${prefix}gripper_r_link2"/>
 	<child link="${prefix}gripper_r_link_finger"/>
-        <origin xyz="0.0 0.053 0.0" rpy="${PI} 0 ${PI}"/>
+	<origin xyz="0.0 0.053 0.0" rpy="${PI} 0 ${PI}"/>
 	<axis xyz="0 0 1" />
 	<limit lower="-10" upper="10" effort="100" velocity="1" />
 </joint>
-<joint name="${prefix}gripper_l_joint1" type="revolute">
+<joint name="${prefix}gripper_l_joint1" type="fixed">
 	<parent link="${prefix}gripper_base_link"/>
 	<child link="${prefix}gripper_l_link1"/>
@@ -145,15 +145,15 @@
 	<limit lower="-10.0" upper="10.0" effort="100" velocity="1" />
 </joint>
-<joint name="${prefix}gripper_l_joint2" type="revolute">
+<joint name="${prefix}gripper_l_joint2" type="fixed">
 	<parent link="${prefix}gripper_base_link"/>
 	<child link="${prefix}gripper_l_link2"/>
-        <origin xyz="-0.0115 0.0 0.1056" rpy="${PI_2} 0 ${PI}"/>
+	<origin xyz="-0.0115 0.0 0.1056" rpy="${PI_2} 0 ${PI}"/>
 	<axis xyz="0 0 1" />
 	<limit lower="-10.0" upper="10.0" effort="100" velocity="1" />
 </joint>
-<joint name="${prefix}gripper_l_joint_finger" type="revolute">
+<joint name="${prefix}gripper_l_joint_finger" type="fixed">
 	<parent link="${prefix}gripper_l_link2"/>
 	<child link="${prefix}gripper_l_link_finger"/>
-        <origin xyz="0.0 0.053 0.0" rpy="${PI} 0 ${PI}"/>
+	<origin xyz="0.0 0.053 0.0" rpy="${PI} 0 ${PI}"/>
 	<axis xyz="0 0 1" />
 	<limit lower="-10" upper="10" effort="100" velocity="1" />

Commit message: c

File: lebai_lm3_support/urdf/gripper_macro.xacro (robot description, xacro)
@@ -117,5 +117,5 @@
 <!-- end of link list -->
 <!-- joint list -->
-<joint name="${prefix}gripper_r_joint1" type="fixed">
+<joint name="${prefix}gripper_r_joint1" type="revolute">
 	<parent link="${prefix}gripper_base_link"/>
 	<child link="${prefix}gripper_r_link1"/>
@@ -124,5 +124,5 @@
 	<limit lower="-10.0" upper="10.0" effort="100" velocity="1" />
 </joint>
-<joint name="${prefix}gripper_r_joint2" type="fixed">
+<joint name="${prefix}gripper_r_joint2" type="revolute">
 	<parent link="${prefix}gripper_base_link"/>
 	<child link="${prefix}gripper_r_link2"/>
@@ -131,5 +131,5 @@
 	<limit lower="-10.0" upper="10.0" effort="100" velocity="1" />
 </joint>
-<joint name="${prefix}gripper_r_joint_finger" type="fixed">
+<joint name="${prefix}gripper_r_joint_finger" type="revolute">
 	<parent link="${prefix}gripper_r_link2"/>
 	<child link="${prefix}gripper_r_link_finger"/>
@@ -138,5 +138,5 @@
 	<limit lower="-10" upper="10" effort="100" velocity="1" />
 </joint>
-<joint name="${prefix}gripper_l_joint1" type="fixed">
+<joint name="${prefix}gripper_l_joint1" type="revolute">
 	<parent link="${prefix}gripper_base_link"/>
 	<child link="${prefix}gripper_l_link1"/>
@@ -145,5 +145,5 @@
 	<limit lower="-10.0" upper="10.0" effort="100" velocity="1" />
 </joint>
-<joint name="${prefix}gripper_l_joint2" type="fixed">
+<joint name="${prefix}gripper_l_joint2" type="revolute">
 	<parent link="${prefix}gripper_base_link"/>
 	<child link="${prefix}gripper_l_link2"/>
@@ -152,5 +152,5 @@
 	<limit lower="-10.0" upper="10.0" effort="100" velocity="1" />
 </joint>
-<joint name="${prefix}gripper_l_joint_finger" type="fixed">
+<joint name="${prefix}gripper_l_joint_finger" type="revolute">
 	<parent link="${prefix}gripper_l_link2"/>
 	<child link="${prefix}gripper_l_link_finger"/>

Commit message: p

File: lebai_lm3_support/urdf/gripper_macro.xacro (robot description, xacro)
@@ -115,4 +115,5 @@
 </link>
 <link name="${prefix}gripper_tip" />
+<link name="${prefix}end_effector" />
 <!-- end of link list -->
 <!-- joint list -->

File: lebai_lm3_support/urdf/lm3_with_gripper.xacro (robot description, xacro)
@@ -14,3 +14,8 @@
     	<child link="gripper_base_link"/>
   	</joint>
+	<joint name="tool0_to_end_effector_joint" type="fixed">
+		<parent link="tool0"/>
+		<child link="end_effector"/>
+		<origin xyz="0.0 0.0 0.17" rpy="0.0 0.0 0.0"/>
+	</joint>
 </robot>
